Commit message: Added rplidar

File: novel_gazebo/model/turtlebot_lidar/sensors/lidar.urdf.xacro (robot description, xacro)
@@ -10,5 +10,5 @@
       <origin xyz="0 0 0.0" rpy="0 0 0"/>
       <geometry>
-        <mesh filename="package://turtlebot3_description/meshes/sensors/lds.stl" scale="0.001 0.001 0.001"/>
+        <mesh filename="package://novel_gazebo/model/turtlebot_lidar/mesh/rplidar-a2m4-r1.stl" scale="0.001 0.001 0.001"/>
       </geometry>
       <material name="dark"/>
@@ -31,5 +31,5 @@
     <parent link="base_link"/>
     <child link="base_scan"/>
-    <origin xyz="0 0 0.220841" rpy="0 0 0"/>
+    <origin xyz="0 0 0.19" rpy="0 0 0"/>
   </joint>
   <gazebo reference="base_scan">
@@ -48,5 +48,5 @@
         </scan>
         <range>
-          <min>0.120</min>
+          <min>0.20</min>
           <max>3.5</max>
           <resolution>0.015</resolution>

Commit message: Updated laser frame, more accurate size calculations

File: novel_gazebo/model/turtlebot_lidar/sensors/lidar.urdf.xacro (robot description, xacro)
@@ -31,10 +31,10 @@
     <parent link="base_link"/>
     <child link="base_scan"/>
-    <origin xyz="0 0 0.19" rpy="0 0 0"/>
+    <origin xyz="0 0 0.19" rpy="0 0 ${pi}"/>
   </joint>
   <gazebo reference="base_scan">
     <material>Gazebo/FlatBlack</material>
     <sensor type="ray" name="lds_lfcd_sensor">
-      <pose>0 0 0 0 0 0</pose>
+      <pose>0 0 0 0 0 3.14159</pose>
       <update_rate>5</update_rate>
       <ray>
